File: Schaltplan/CallForHelp.brd (EAGLE design)
At the start: 76.5 x 60.2 mm, 20 parts

Commit message: updated versions
Parts:
- added R6: 100kΩ, rcl:0204/7
- moved R1 13.0 mm to (25.5, 33.6)
- moved BATTERIE 5.30 mm to (11.5, 14.2)
- moved WEMOS1 3.26 mm to (11.9, 34.5)
Connections:
- new net N$5: R6.1, WEMOS1.A0
- net V+: now also R6.2
Routing:
- net V+: track 89.0 -> 134.8 mm
- net N$5: track 0.00 -> 36.5 mm, vias 0 -> 1
- net LED_PIN: track 32.9 -> 19.4 mm
- net N$3: track 3.05 -> 12.7 mm
- net BATTERY_GND: track 31.5 -> 36.8 mm
- net BATTERY_VCC: track 31.4 -> 36.7 mm
- net N$7: track 34.2 -> 30.7 mm
- net N$6: track 34.2 -> 30.8 mm
- net N$8: track 34.9 -> 31.6 mm
- net GND: track 155.1 -> 158.1 mm
- net +5V: track 67.9 -> 70.8 mm
Other:
- board size 76.5 x 60.2 mm -> 76.3 x 56.8 mm
