File: Schaltplan/CallForHelp.sch (EAGLE design)
At the start: 20 parts

Commit message: updated versions
Parts:
- added R6: 100kΩ, rcl:R-EU_0204/7
Connections:
- new net N$5: R6.1, WEMOS1.A0
- net V+: now also R6.2
Other:
- moved on the sheet: C1, R1, SWITCH, WEMOS1
